File: hardware/cf/cfmodule.brd (EAGLE design)
At the start: 59.1 x 73 mm, 13 parts

Commit message: CF module updated
Parts:
- removed C2: (no value), rcl:C0603
- removed E$4: (no value), 74xx-eu:SO20W
- removed R1: (no value), rcl:0204/7
- moved C24 32.0 mm to (30.9, 20.0), turned to 180 degrees
- moved E$2 8.25 mm to (28.6, 5.08)
- moved C1 7.62 mm to (39.2, 28.9)
- moved E$3 6.98 mm to (45.7, 21.0)
Connections:
- removed net IN_A0: E$2.14, E$4.3
- removed net IN_A1: E$2.15, E$4.4
- removed net IN_A2: E$2.16, E$4.5
- removed net IN_CF_CS0: E$2.27, E$3.19, E$4.19, E$4.9
- removed net IN_IO_RD: E$2.26, E$3.1, E$4.8
- removed net IN_IO_WR: E$2.25, E$4.7
- removed net IN_RST: E$2.18, E$4.6
- removed net S$4: E$4.1, R1.1
- net A0: now also E$2.14; no longer E$4.17
- net A1: now also E$2.15; no longer E$4.16
- net A2: now also E$2.16; no longer E$4.15
- net CF_CS0: now also E$2.27, E$3.19; no longer E$4.11
- net GND: no longer C2.2, E$4.10, E$4.2
- net IO_RD: now also E$2.26, E$3.1; no longer E$4.12
- net IO_WR: now also E$2.25; no longer E$4.13
- net RST: now also E$2.18; no longer E$4.14
- net VCC: no longer C2.1, E$4.20, R1.2
Routing:
- net IN_CF_CS0: track 73.3 -> 0.00 mm, vias 2 -> 0
- net VCC: track 143.1 -> 93.4 mm, vias 4 -> 2
- net GND: track 108.5 -> 82.4 mm, vias 8 -> 0
- net CF_CS0: track 24.2 -> 49.7 mm
- net IO_RD: track 24.2 -> 44.6 mm, vias 0 -> 2
- net IN_IO_RD: track 20.4 -> 0.00 mm, vias 2 -> 0
- net S$9: track 64.1 -> 45.2 mm, vias 0 -> 2
- net IO_WR: track 24.2 -> 41.2 mm
- net IN_A1: track 15.8 -> 0.00 mm
- net IN_IO_WR: track 15.8 -> 0.00 mm
- net A1: track 27.1 -> 40.7 mm
- net IN_A2: track 12.7 -> 0.00 mm
- net IN_A0: track 12.7 -> 0.00 mm
- net IN_RST: track 12.2 -> 0.00 mm
- net RST: track 26.8 -> 37.6 mm
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Other:
- board size 59.1 x 73 mm -> 59.1 x 64.8 mm
