File: hardware/cpu/cpu_board.sch (EAGLE design)
At the start: 53 parts, among them IC4 7404N, IC5 7400N, IC6 74HCT139N, IC7 7400N, IC9 74HCT138N, X1 22-23-2041

Commit message: Bug in memory address decoder fixed
Connections:
- removed net !A15: IC4A.O, IC6A.G
- new net CS_RAM: IC6A.Y0, U$4.!CS
- net A13: no longer IC6B.A
- net A14: now also IC6B.A; no longer IC6A.A
- net A15: now also IC6A.A; no longer IC4A.I, U$4.!CS
- net CS_EPROM: now also IC6B.Y1; no longer IC6A.Y1
- net GND: now also IC4A.I, IC6A.G
- net N$19: now also IC6A.Y1; no longer IC6A.Y0
Other:
- moved on the sheet: IC4A

Commit message: AEN signal connected to memory address decoder
Connections:
- net AEN: now also IC6A.G
- net GND: no longer IC6A.G
Changed lines of the file:
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@@
 <pinref part="GND10" gate="1" pin="GND"/>
 <wire x1="10.16" y1="-147.32" x2="7.62" y2="-147.32" width="0.1524" layer="91"/>
-<wire x1="7.62" y1="-147.32" x2="7.62" y2="-152.4" width="0.1524" layer="91"/>
-<pinref part="IC6" gate="A" pin="G"/>
-<wire x1="7.62" y1="-152.4" x2="7.62" y2="-157.48" width="0.1524" layer="91"/>
-<wire x1="10.16" y1="-152.4" x2="7.62" y2="-152.4" width="0.1524" layer="91"/>
-<junction x="7.62" y="-152.4"/>
+<wire x1="7.62" y1="-147.32" x2="7.62" y2="-157.48" width="0.1524" layer="91"/>
 </segment>
 <segment>
@@
 <wire x1="116.84" y1="-147.32" x2="114.3" y2="-147.32" width="0.1524" layer="91"/>
 </segment>
-</net>
+<segment>
+<pinref part="IC6" gate="A" pin="G"/>
+<wire x1="10.16" y1="-152.4" x2="2.54" y2="-152.4" width="0.1524" layer="91"/>
+<label x="2.54" y="-152.4" size="1.4224" layer="95" rot="R180" xref="yes"/>
+</segment>
+</net>

Commit message: AEN removed from memory address decoder
Connections:
- net AEN: no longer IC6A.G
- net GND: now also IC6A.G
Changed lines of the file:
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@@
 <pinref part="GND10" gate="1" pin="GND"/>
 <wire x1="10.16" y1="-147.32" x2="7.62" y2="-147.32" width="0.1524" layer="91"/>
-<wire x1="7.62" y1="-147.32" x2="7.62" y2="-157.48" width="0.1524" layer="91"/>
+<wire x1="7.62" y1="-147.32" x2="7.62" y2="-152.4" width="0.1524" layer="91"/>
+<pinref part="IC6" gate="A" pin="G"/>
+<wire x1="7.62" y1="-152.4" x2="7.62" y2="-157.48" width="0.1524" layer="91"/>
+<wire x1="10.16" y1="-152.4" x2="7.62" y2="-152.4" width="0.1524" layer="91"/>
+<junction x="7.62" y="-152.4"/>
 </segment>
 <segment>
@@
 <wire x1="116.84" y1="-147.32" x2="114.3" y2="-147.32" width="0.1524" layer="91"/>
 </segment>
-<segment>
-<pinref part="IC6" gate="A" pin="G"/>
-<wire x1="10.16" y1="-152.4" x2="2.54" y2="-152.4" width="0.1524" layer="91"/>
-<label x="2.54" y="-152.4" size="1.4224" layer="95" rot="R180" xref="yes"/>
-</segment>
-</net>
+</net>
