File: hardware/cpu_rom_shadowing/cpu_board.sch (EAGLE design)
At the start: 53 parts, among them IC4 7404N, IC5 7400N, IC6 74HCT139N, IC7 7400N, IC9 74HCT138N, X1 22-23-2041

Commit message: ROM shadowed version of PCB modified
Parts:
- removed C15: 100n, rcl:C-EUC1206
- removed C5: 100n, rcl:C-EUC0603
- removed IC4: 7404N, 74xx-us:7404N
- removed IC7: 7400N, 74xx-eu:7400N
- IC5: value 7400N -> 74HCT08N; device 74xx-eu:7400N -> 74xx-eu:74HCT08N
Connections:
- removed net A14_SWITCH: IC5B.O, U$5.DI6
- removed net A15_SWITCH: IC5A.O, U$5.DI2
- removed net BANK_A14: IC7B.O, U$2.A14
- removed net CS_BANKED_RAM: IC6B.Y0, U$2.!CS
- removed net CS_RAM: IC6A.Y0, U$4.!CS
- removed net N$19: IC6A.Y1, IC6B.G
- removed net N$20: IC9A.G1, R9.1
- removed net N$21: IC5B.I1, IC5C.O
- removed net N$26: IC5A.I0, IC5D.O
- removed net START_MEM_SWITCH: IC5A.I1, IC5B.I0, U$1.DO2
- new net CS_RAM1: IC6B.Y2, U$4.!CS
- new net CS_RAM2: IC5B.O, U$2.!CS
- new net N$2: IC5B.I0, IC6B.Y1
- new net N$8: IC5B.I1, IC6B.Y3
- new net PULLUP_5V: IC5C.I1, IC5D.I0, IC9A.G1, R9.1
- new net SHADOW_ROM: IC6B.A, U$1.DO2
- net !CS_PORT_OUT: now also IC5C.O; no longer IC4D.O
- net !RESET: now also IC5D.O; no longer IC4B.O
- net 8275_DACK: no longer IC7B.I0
- net A14: now also U$2.A14; no longer IC6B.A
- net A14_CPU: now also U$5.DI6; no longer IC5C.I0, IC5C.I1
- net A15: now also IC6B.B; no longer IC6A.A
- net A15_CPU: now also U$5.DI2; no longer IC5D.I0, IC5D.I1
- net CS_EPROM: now also IC6B.Y0; no longer IC6B.Y1
- net CS_PORT_OUT: now also IC5C.I0; no longer IC4D.I
- net GND: now also IC5A.I0, IC5A.I1, IC6A.A, IC6B.G; no longer C15.2, C5.2, IC4A.I, IC4C.I, IC4E.I, IC4F.I, IC4P.GND, IC6B.B, IC7A.I0, IC7A.I1, IC7C.I0, IC7C.I1, IC7D.I0, IC7D.I1, IC7P.GND
- net RESET: now also IC5D.I1; no longer IC4B.I
- net SET_BANK_A14: no longer IC7B.I1
- net VCC: no longer C15.1, C5.1, IC4P.VCC, IC7P.VCC
Other:
- moved on the sheet: C10, C16, C23, IC6A, IC6B

Commit message: CPU board (ROM shadowing version) fix
Parts:
- IC5: value 74HCT08N -> 74LS86N; device 74xx-eu:74HCT08N -> 74xx-us:74LS86N
Connections:
- new net N$16: IC5B.I1, IC6A.Y3
- net A15: now also IC6B.A; no longer IC6B.B
- net GND: no longer IC6A.A, IC6A.B
- net N$2: now also IC6A.A; no longer IC5B.I0
- net N$8: now also IC6A.B; no longer IC5B.I1
- net PULLUP_5V: now also IC5B.I0
- net SHADOW_ROM: now also IC6B.B; no longer IC6B.A
Other:
- moved on the sheet: IC6A
Changed lines of the file:
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@@
 <part name="SV2" library="con-harting-ml" deviceset="ML64" device="L"/>
 <part name="GND28" library="supply1" deviceset="GND" device=""/>
-<part name="IC5" library="74xx-eu" deviceset="74*08" device="N" technology="HCT"/>
+<part name="IC5" library="74xx-us" deviceset="74*86" device="N" technology="LS"/>
 </parts>
 <sheets>
@@
 <instance part="IC6" gate="B" x="-30.48" y="-147.32"/>
 <instance part="GND10" gate="1" x="-45.72" y="-160.02"/>
-<instance part="GND11" gate="1" x="-45.72" y="-193.04"/>
+<instance part="GND11" gate="1" x="2.54" y="-162.56"/>
 <instance part="GND12" gate="1" x="114.3" y="-160.02"/>
 <instance part="R9" gate="G$1" x="101.6" y="-137.16" rot="R90"/>
@@
 <instance part="SV2" gate="1" x="152.4" y="-33.02"/>
 <instance part="GND28" gate="1" x="-40.64" y="88.9"/>
-<instance part="IC5" gate="B" x="10.16" y="-149.86"/>
+<instance part="IC5" gate="B" x="55.88" y="-152.4"/>
 <instance part="IC5" gate="C" x="215.9" y="-152.4"/>
 <instance part="IC5" gate="D" x="215.9" y="-132.08"/>
 <instance part="IC5" gate="P" x="50.8" y="-111.76"/>
-<instance part="IC6" gate="A" x="-27.94" y="-180.34"/>
+<instance part="IC6" gate="A" x="20.32" y="-149.86"/>
 <instance part="IC5" gate="A" x="215.9" y="-213.36"/>
 </instances>
@@
 <segment>
 <pinref part="GND11" gate="1" pin="GND"/>
-<wire x1="-45.72" y1="-177.8" x2="-45.72" y2="-180.34" width="0.1524" layer="91"/>
-<pinref part="IC6" gate="A" pin="A"/>
-<wire x1="-45.72" y1="-180.34" x2="-45.72" y2="-185.42" width="0.1524" layer="91"/>
-<wire x1="-45.72" y1="-185.42" x2="-45.72" y2="-190.5" width="0.1524" layer="91"/>
-<wire x1="-40.64" y1="-177.8" x2="-45.72" y2="-177.8" width="0.1524" layer="91"/>
-<pinref part="IC6" gate="A" pin="B"/>
-<wire x1="-40.64" y1="-180.34" x2="-45.72" y2="-180.34" width="0.1524" layer="91"/>
-<junction x="-45.72" y="-180.34"/>
+<wire x1="2.54" y1="-154.94" x2="2.54" y2="-160.02" width="0.1524" layer="91"/>
 <pinref part="IC6" gate="A" pin="G"/>
-<wire x1="-40.64" y1="-185.42" x2="-45.72" y2="-185.42" width="0.1524" layer="91"/>
-<junction x="-45.72" y="-185.42"/>
+<wire x1="7.62" y1="-154.94" x2="2.54" y2="-154.94" width="0.1524" layer="91"/>
 </segment>
 <segment>
@@
 <pinref part="IC5" gate="A" pin="I0"/>
 <wire x1="203.2" y1="-215.9" x2="203.2" y2="-223.52" width="0.1524" layer="91"/>
-<wire x1="208.28" y1="-210.82" x2="203.2" y2="-210.82" width="0.1524" layer="91"/>
 <pinref part="IC5" gate="A" pin="I1"/>
-<wire x1="208.28" y1="-215.9" x2="203.2" y2="-215.9" width="0.1524" layer="91"/>
 <junction x="203.2" y="-215.9"/>
 </segment>
@@
 </segment>
 <segment>
-<wire x1="-43.18" y1="-147.32" x2="-45.72" y2="-147.32" width="0.1524" layer="91"/>
-<label x="-45.72" y="-147.32" size="1.4224" layer="95" rot="R180" xref="yes"/>
-<pinref part="IC6" gate="B" pin="B"/>
+<wire x1="-43.18" y1="-144.78" x2="-45.72" y2="-144.78" width="0.1524" layer="91"/>
+<label x="-45.72" y="-144.78" size="1.4224" layer="95" rot="R180" xref="yes"/>
+<pinref part="IC6" gate="B" pin="A"/>
 </segment>
 </net>
@@
 </segment>
 <segment>
-<wire x1="17.78" y1="-149.86" x2="25.4" y2="-149.86" width="0.1524" layer="91"/>
 <pinref part="IC5" gate="B" pin="O"/>
+<wire x1="68.58" y1="-152.4" x2="73.66" y2="-152.4" width="0.1524" layer="91"/>
+<label x="73.66" y="-152.4" size="1.4224" layer="95" xref="yes"/>
 </segment>
 </net>
@@
 <segment>
 <pinref part="IC5" gate="C" pin="I1"/>
-<wire x1="208.28" y1="-154.94" x2="200.66" y2="-154.94" width="0.1524" layer="91"/>
+<wire x1="203.2" y1="-154.94" x2="200.66" y2="-154.94" width="0.1524" layer="91"/>
 <label x="200.66" y="-154.94" size="1.4224" layer="95" rot="R180" xref="yes"/>
 </segment>
 <segment>
 <pinref part="IC5" gate="D" pin="I0"/>
-<wire x1="208.28" y1="-129.54" x2="200.66" y2="-129.54" width="0.1524" layer="91"/>
+<wire x1="203.2" y1="-129.54" x2="200.66" y2="-129.54" width="0.1524" layer="91"/>
+<label x="200.66" y="-129.54" size="1.4224" layer="95" rot="R180" xref="yes"/>
+</segment>
+<segment>
+<wire x1="43.18" y1="-149.86" x2="40.64" y2="-149.86" width="0.1524" layer="91"/>
+<pinref part="IC5" gate="B" pin="I0"/>
+<wire x1="40.64" y1="-149.86" x2="40.64" y2="-142.24" width="0.1524" layer="91"/>
+<label x="40.64" y="-142.24" size="1.4224" layer="95" rot="R90" xref="yes"/>
 </segment>
 </net>
@@
 </segment>
 <segment>
-<wire x1="208.28" y1="-149.86" x2="200.66" y2="-149.86" width="0.1524" layer="91"/>
+<wire x1="203.2" y1="-149.86" x2="200.66" y2="-149.86" width="0.1524" layer="91"/>
 <label x="200.66" y="-149.86" size="1.4224" layer="95" rot="R180" xref="yes"/>
 <pinref part="IC5" gate="C" pin="I0"/>
@@
 </segment>
 <segment>
-<wire x1="208.28" y1="-134.62" x2="200.66" y2="-134.62" width="0.1524" layer="91"/>
+<wire x1="203.2" y1="-134.62" x2="200.66" y2="-134.62" width="0.1524" layer="91"/>
 <label x="200.66" y="-134.62" size="1.4224" layer="95" rot="R180" xref="yes"/>
 <pinref part="IC5" gate="D" pin="I1"/>
@@
 </segment>
 <segment>
-<wire x1="223.52" y1="-132.08" x2="228.6" y2="-132.08" width="0.1524" layer="91"/>
 <label x="228.6" y="-132.08" size="1.4224" layer="95" xref="yes"/>
 <pinref part="IC5" gate="D" pin="O"/>
@@
 <net name="!CS_PORT_OUT" class="0">
 <segment>
-<wire x1="223.52" y1="-152.4" x2="228.6" y2="-152.4" width="0.1524" layer="91"/>
 <label x="228.6" y="-152.4" size="1.4224" layer="95" xref="yes"/>
 <pinref part="IC5" gate="C" pin="O"/>
@@
 <net name="SHADOW_ROM" class="0">
 <segment>
-<wire x1="-43.18" y1="-144.78" x2="-45.72" y2="-144.78" width="0.1524" layer="91"/>
-<label x="-45.72" y="-144.78" size="1.4224" layer="95" rot="R180" xref="yes"/>
-<pinref part="IC6" gate="B" pin="A"/>
-</segment>
-<segment>
 <pinref part="U$1" gate="G$1" pin="DO2"/>
 <wire x1="358.14" y1="45.72" x2="363.22" y2="45.72" width="0.1524" layer="91"/>
 <label x="363.22" y="45.72" size="1.4224" layer="95" xref="yes"/>
 </segment>
+<segment>
+<pinref part="IC6" gate="B" pin="B"/>
+<wire x1="-43.18" y1="-147.32" x2="-45.72" y2="-147.32" width="0.1524" layer="91"/>
+<label x="-45.72" y="-147.32" size="1.4224" layer="95" rot="R180" xref="yes"/>
+</segment>
 </net>
 <net name="N$2" class="0">
 <segment>
-<wire x1="2.54" y1="-147.32" x2="-17.78" y2="-147.32" width="0.1524" layer="91"/>
 <pinref part="IC6" gate="B" pin="Y1"/>
-<pinref part="IC5" gate="B" pin="I0"/>
+<pinref part="IC6" gate="A" pin="A"/>
+<wire x1="-17.78" y1="-147.32" x2="7.62" y2="-147.32" width="0.1524" layer="91"/>
 </segment>
 </net>
 <net name="N$8" class="0">
 <segment>
-<wire x1="2.54" y1="-152.4" x2="-17.78" y2="-152.4" width="0.1524" layer="91"/>
 <pinref part="IC6" gate="B" pin="Y3"/>
+<pinref part="IC6" gate="A" pin="B"/>
+<wire x1="7.62" y1="-149.86" x2="2.54" y2="-149.86" width="0.1524" layer="91"/>
+<wire x1="-17.78" y1="-152.4" x2="2.54" y2="-152.4" width="0.1524" layer="91"/>
+<wire x1="2.54" y1="-152.4" x2="2.54" y2="-149.86" width="0.1524" layer="91"/>
+</segment>
+</net>
+<net name="N$16" class="0">
+<segment>
 <pinref part="IC5" gate="B" pin="I1"/>
-</segment>
-</net>
+<pinref part="IC6" gate="A" pin="Y3"/>
+<wire x1="33.02" y1="-154.94" x2="43.18" y2="-154.94" width="0.1524" layer="91"/>
+</segment>
+</net>
