File: hardware/cpu_ultra/cpu_board.brd (EAGLE design)
At the start: 148.6 x 122.5 mm, 41 parts, among them IC5 74AC157N, IC6 74AC273N, IC9 74HCT138N, U1 AS6C4008-55PCN, X1 22-23-2041

Commit message: ULTRA CPU board updatye
Parts:
- added C3: (no value), rcl:C0603
- added IC11: 74LVC1G08DBV, 74xx-little-de:SOT23-5
- added IC7: 7402N, 74xx-eu:DIL14
- C14, C9: device rcl:C1206 -> rcl:C0603
- moved C14 114.5 mm to (94.5, 98.4)
- moved C12 50.6 mm to (76.8, 10.8), turned to 0 degrees
- moved C9 8.21 mm to (94.5, 109.9), turned to 0 degrees
- moved C10 5.43 mm to (124.5, 111.8), turned to 90 degrees
- moved C19 4.45 mm to (91.4, 104.3)
- moved JP1 4.44 mm to (90.2, 101.0)
- moved R9 1.42 mm to (124.8, 11.4)
- moved C13 1.27 mm to (115.9, 18.7)
- moved IC9 1.27 mm to (124.8, 11.4)
Connections:
- new net N$2: IC11.4, IC5.1
- new net PORT_OUT_WR: IC6.11, IC7.10
- net !RESET: now also IC7.1
- net A14: now also IC11.2
- net A15: now also IC11.1
- net A19_CS_EPROM: now also IC7.11, IC7.12
- net CS_PORT_OUT: now also IC7.8; no longer IC6.11
- net CS_RAM1: now also IC7.13
- net GND: now also C3.2, IC11.3, IC7.5, IC7.6, IC7.7
- net IO_WR: now also IC7.9
- net RESET: now also IC7.2, IC7.3
- net VCC: now also C3.1, IC11.5, IC7.14
Routing:
- net VCC: track 422.6 -> 568.2 mm
- net PORT_OUT_WR: track 0.00 -> 120.5 mm, vias 0 -> 2
- net A19_CS_EPROM: track 85.2 -> 161.8 mm, vias 2 -> 4
- net N$2: track 0.00 -> 56.5 mm
- net A14: track 124.0 -> 164.8 mm
- net A15: track 170.3 -> 210.1 mm
- net CS_PORT_OUT: track 0.00 -> 39.4 mm, vias 0 -> 2
- net RESET: track 207.4 -> 239.5 mm, vias 2 -> 4
- net GND: track 142.2 -> 162.9 mm, vias 16 -> 20
- net IO_WR: track 125.1 -> 141.0 mm, vias 2 -> 4
- net !RESET: track 162.2 -> 153.9 mm
- net CS_RAM1: track 71.0 -> 77.9 mm, vias 1 -> 2
- net N$12: track 21.2 -> 16.8 mm
- net A6: track 267.9 -> 270.7 mm
- net OUT_4: track 1.80 -> 0.00 mm
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Other:
- board text added: "POLON ULTRA CPU BOARD RQ9RZI 2025"
