File: hardware/cpu_ultra/cpu_board.brd (EAGLE design)
At the start: 148.6 x 122.5 mm, 44 parts, among them IC11 74LVC1G08DBV, IC5 74AC157N, IC6 74AC273N, IC7 7402N, IC9 74HCT138N, U1 AS6C4008-55PCN, X1 22-23-2041

Commit message: Bug fixed
Connections:
- removed net N$42: IC4.24
- net RD: now also IC4.24
Routing:
- net A3: track 202.9 -> 212.6 mm
- net RD: track 145.7 -> 155.0 mm
Changed lines of the file:
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@@
 <wire x1="35.56" y1="93.345" x2="35.56" y2="43.18" width="0.4064" layer="1"/>
 <via x="35.56" y="43.18" extent="1-16" drill="0.6" diameter="1.4224" shape="octagon"/>
-<via x="76.2" y="38.1" extent="1-16" drill="0.6" diameter="1.4224" shape="octagon"/>
-<via x="76.2" y="65.405" extent="1-16" drill="0.6" diameter="1.4224" shape="octagon"/>
-<wire x1="76.2" y1="65.405" x2="76.2" y2="38.1" width="0.4064" layer="1"/>
+<via x="98.425" y="38.1" extent="1-16" drill="0.6" diameter="1.4224" shape="octagon"/>
+<via x="98.425" y="66.675" extent="1-16" drill="0.6" diameter="1.4224" shape="octagon"/>
+<wire x1="98.425" y1="66.675" x2="98.425" y2="38.1" width="0.4064" layer="1"/>
 <contactref element="SV2" pad="18"/>
 <contactref element="U1" pad="9"/>
 <contactref element="IC4" pad="9"/>
 <wire x1="109.855" y1="66.675" x2="127" y2="66.675" width="0.4064" layer="16"/>
-<wire x1="97.155" y1="66.675" x2="109.855" y2="66.675" width="0.4064" layer="16"/>
-<wire x1="76.2" y1="65.405" x2="85.725" y2="65.405" width="0.4064" layer="16"/>
-<wire x1="85.725" y1="65.405" x2="86.995" y2="66.675" width="0.4064" layer="16"/>
-<wire x1="86.995" y1="66.675" x2="89.535" y2="66.675" width="0.4064" layer="16"/>
+<wire x1="86.995" y1="66.675" x2="89.535" y2="66.675" width="0" layer="19" extent="1-16"/>
 <wire x1="35.56" y1="43.18" x2="68.8975" y2="43.18" width="0.4064" layer="16"/>
 <wire x1="68.8975" y1="43.18" x2="73.9775" y2="38.1" width="0.4064" layer="16"/>
-<wire x1="73.9775" y1="38.1" x2="76.2" y2="38.1" width="0.4064" layer="16"/>
+<wire x1="73.9775" y1="38.1" x2="98.425" y2="38.1" width="0.4064" layer="16"/>
+<wire x1="97.155" y1="66.675" x2="98.425" y2="66.675" width="0.4064" layer="16"/>
+<wire x1="98.425" y1="66.675" x2="109.855" y2="66.675" width="0.4064" layer="16"/>
 </signal>
 <signal name="A4">
@@
 <wire x1="102.235" y1="59.055" x2="109.855" y2="59.055" width="0.4064" layer="16"/>
 <wire x1="109.855" y1="59.055" x2="118.745" y2="59.055" width="0.4064" layer="16"/>
-<wire x1="102.235" y1="5.715" x2="117.475" y2="5.715" width="0.4064" layer="16"/>
 <wire x1="117.475" y1="5.715" x2="118.4275" y2="6.6675" width="0.4064" layer="16"/>
 <wire x1="118.4275" y1="7.62" x2="118.4275" y2="6.6675" width="0.4064" layer="16"/>
+<wire x1="102.235" y1="5.715" x2="117.475" y2="5.715" width="0.4064" layer="16"/>
 </signal>
 <signal name="A7">
@@
 <contactref element="U1" pad="24"/>
 <wire x1="85.09" y1="21.59" x2="108.585" y2="21.59" width="0.4064" layer="16"/>
-<wire x1="74.295" y1="66.675" x2="85.09" y2="66.675" width="0.4064" layer="16"/>
-<via x="85.09" y="66.675" extent="1-16" drill="0.6" diameter="1.4224" shape="octagon"/>
-<wire x1="85.09" y1="66.675" x2="85.09" y2="21.59" width="0.4064" layer="1"/>
+<via x="85.09" y="65.405" extent="1-16" drill="0.6" diameter="1.4224" shape="octagon"/>
+<wire x1="85.09" y1="65.405" x2="85.09" y2="21.59" width="0.4064" layer="1"/>
+<contactref element="IC4" pad="24"/>
+<wire x1="85.09" y1="65.405" x2="91.44" y2="65.405" width="0.4064" layer="16"/>
+<wire x1="91.44" y1="65.405" x2="92.71" y2="66.675" width="0.4064" layer="16"/>
+<wire x1="92.71" y1="66.675" x2="94.615" y2="66.675" width="0.4064" layer="16"/>
+<wire x1="85.09" y1="65.405" x2="76.835" y2="65.405" width="0.4064" layer="16"/>
+<wire x1="76.835" y1="65.405" x2="75.565" y2="66.675" width="0.4064" layer="16"/>
+<wire x1="75.565" y1="66.675" x2="74.295" y2="66.675" width="0.4064" layer="16"/>
 </signal>
 <signal name="IO_RD">
@@
 <wire x1="117.475" y1="79.375" x2="117.475" y2="86.0425" width="0.4064" layer="1"/>
 </signal>
-<signal name="N$42">
-<contactref element="IC4" pad="24"/>
-</signal>
 <signal name="A19_CS_EPROM">

Commit message: Several bugs fixed
Parts:
- moved C7 11.8 mm to (56.5, 118.7), turned to 180 degrees
Routing:
- net GND: track 162.9 -> 158.4 mm
- net NEG_5V: track 60.9 -> 64.4 mm
- net VCC: track 568.2 -> 567.5 mm
Changed lines of the file:
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@@
 </element>
 <element name="C24" library="rcl" package="E3,5-8" value="" x="20.955" y="116.205" rot="R180"/>
-<element name="C7" library="rcl" package="E2,5-7" value="" x="44.7675" y="117.475" rot="R90"/>
+<element name="C7" library="rcl" package="E2,5-7" value="" x="56.515" y="118.745" rot="R180"/>
 <element name="SV2" library="con-harting-ml" package="ML64L" value="" x="137.4775" y="56.515" rot="R270">
 <attribute name="OC_NEWARK" value="unknown" x="137.4775" y="56.515" size="1.778" layer="27" rot="R270" display="off"/>
@@
 <wire x1="49.2125" y1="48.898" x2="67.6245" y2="48.898" width="1.27" layer="16"/>
 <wire x1="67.6245" y1="48.898" x2="70.1675" y2="46.355" width="1.27" layer="16"/>
-<wire x1="74.292" y1="43.815" x2="74.295" y2="44.453" width="1.27" layer="16"/>
 <wire x1="74.295" y1="44.453" x2="74.295" y2="46.355" width="1.27" layer="16"/>
 <contactref element="IC6" pad="20"/>
@@
 <contactref element="C3" pad="2"/>
 <via x="132.3975" y="93.345" extent="1-16" drill="0.6" diameter="1.4224" shape="octagon"/>
-<via x="132.3975" y="111.125" extent="1-16" drill="0.6" diameter="1.4224" shape="octagon"/>
-<wire x1="132.3975" y1="93.345" x2="132.3975" y2="111.125" width="0.6096" layer="1"/>
+<via x="132.3975" y="106.68" extent="1-16" drill="0.6" diameter="1.4224" shape="octagon"/>
+<wire x1="132.3975" y1="93.345" x2="132.3975" y2="106.68" width="0.6096" layer="1"/>
 <via x="99.695" y="118.745" extent="1-16" drill="0.6" diameter="1.4224" shape="octagon"/>
 <via x="99.695" y="113.665" extent="1-16" drill="0.6" diameter="1.4224" shape="octagon"/>
@@
 <contactref element="IC7" pad="5"/>
 <contactref element="IC7" pad="6"/>
-<wire x1="44.7675" y1="113.6625" x2="44.7675" y2="116.205" width="0" layer="19" extent="16-16"/>
 </signal>
 <signal name="D0">
@@
 <contactref element="IC4" pad="9"/>
 <wire x1="109.855" y1="66.675" x2="127" y2="66.675" width="0.4064" layer="16"/>
-<wire x1="86.995" y1="66.675" x2="89.535" y2="66.675" width="0" layer="19" extent="1-16"/>
 <wire x1="35.56" y1="43.18" x2="68.8975" y2="43.18" width="0.4064" layer="16"/>
 <wire x1="68.8975" y1="43.18" x2="73.9775" y2="38.1" width="0.4064" layer="16"/>
@@
 <contactref element="X1" pad="1"/>
 <contactref element="C7" pad="-"/>
-<wire x1="33.655" y1="118.745" x2="44.7675" y2="118.745" width="1.27" layer="16"/>
-<wire x1="44.7675" y1="118.745" x2="51.7525" y2="118.745" width="1.27" layer="16"/>
+<wire x1="33.655" y1="118.745" x2="51.7525" y2="118.745" width="1.27" layer="16"/>
+<wire x1="51.7525" y1="118.745" x2="55.245" y2="118.745" width="1.27" layer="16"/>
 </signal>
 <signal name="!RESET">

Commit message: Minor bug fixed
Routing:
- net GND: track 158.4 -> 159.7 mm
Changed lines of the file:
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@@
 <contactref element="IC3" pad="14"/>
 <contactref element="IC1" pad="8"/>
-<via x="65.0875" y="112.395" extent="1-16" drill="0.6" diameter="1.4224" shape="octagon"/>
+<via x="65.0875" y="113.665" extent="1-16" drill="0.6" diameter="1.4224" shape="octagon"/>
 <via x="65.0875" y="97.155" extent="1-16" drill="0.6" diameter="1.4224" shape="octagon"/>
-<wire x1="65.0875" y1="112.395" x2="65.0875" y2="97.155" width="0.6096" layer="1"/>
+<wire x1="65.0875" y1="113.665" x2="65.0875" y2="97.155" width="0.6096" layer="1"/>
 <contactref element="C18" pad="2"/>
 <contactref element="C19" pad="2"/>
