File: hardware/cpu_ultra/cpu_board.sch (EAGLE design)
At the start: 41 parts, among them IC5 74AC157N, IC6 74AC273N, IC9 74HCT138N, U1 AS6C4008-55PCN, X1 22-23-2041

Commit message: ULTRA CPU board updatye
Parts:
- added C3: (no value), rcl:C-EUC0603
- added IC11: 74LVC1G08DBV, 74xx-little-de:74LVC1G08DBV
- added IC7: 7402N, 74xx-eu:7402N
- C14, C9: device rcl:C-EUC1206 -> rcl:C-EUC0603
Connections:
- new net N$2: IC11A.O, IC5A.!A!/B
- new net PORT_OUT_WR: IC6A.CLK, IC7C.O
- net !RESET: now also IC7A.O
- net A14: now also IC11A.I1
- net A15: now also IC11A.I0
- net A19_CS_EPROM: now also IC7D.I0, IC7D.I1
- net CS_PORT_OUT: now also IC7C.I0; no longer IC6A.CLK
- net CS_RAM1: now also IC7D.O
- net GND: now also C3.2, IC11P.GND, IC7B.I0, IC7B.I1, IC7P.GND
- net IO_WR: now also IC7C.I1
- net RESET: now also IC7A.I0, IC7A.I1
- net VCC: now also C3.1, IC11P.VCC, IC7P.VCC

Commit message: Bug fixed
Connections:
- removed net N$42: IC4.!OE
- net RD: now also IC4.!OE
Changed lines of the file:
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@@
 <label x="243.84" y="-22.86" size="1.4224" layer="95" rot="R180" xref="yes"/>
+</segment>
+<segment>
+<pinref part="IC4" gate="G$1" pin="!OE"/>
+<wire x1="337.82" y1="-60.96" x2="335.28" y2="-60.96" width="0.1524" layer="91"/>
+<label x="335.28" y="-60.96" size="1.4224" layer="95" rot="R180" xref="yes"/>
 </segment>
 </net>
@@
 </segment>
 </net>
-<net name="N$42" class="0">
-<segment>
-<pinref part="IC4" gate="G$1" pin="!OE"/>
-<wire x1="337.82" y1="-60.96" x2="335.28" y2="-60.96" width="0.1524" layer="91"/>
-<label x="335.28" y="-60.96" size="1.4224" layer="95" rot="R180" xref="yes"/>
-</segment>
-</net>
