File: hardware/io_ultra/7880_IO.sch (EAGLE design)
At the start: 64 parts, among them IC11 74HCT245DW, IC4 74HCT139N, IC5 74AC06N, IC7 MAX232, J1 DIN5, X2 CRYSTALS-NOGND-CFPX-217, X3 22-23-2021, X4 CRYSTALS-NOGND-CFPX-217

Commit message: I/O ultra board updated
Parts:
- removed X1: (no value), con-subd:M09HP
- added C11, C28, C29, C30: (no value), rcl:C-EUC0603
- added IC6: MAX232, maxim:MAX232
- added SV1, SV3: (no value), con-ml:ML10
- C2: device rcl:C-EUC1206 -> rcl:C-EUC0603
Connections:
- removed net CTS1: IC7G$1.R2OUT
- removed net N$7: IC7G$1.T2OUT, X1.7
- removed net RTS1: IC7G$1.T2IN
- new net CTS1_TTL: IC2G$1.IP0, IC7G$1.R2OUT
- new net CTS2_TTL: IC2G$1.IP1, IC6G$1.R2OUT
- new net N$15: IC6G$1.T2OUT, SV3.4
- new net N$16: C11.2, IC6G$1.C1+
- new net N$26: C28.2, IC6G$1.C2+
- new net N$27: C28.1, IC6G$1.C2-
- new net N$30: C11.1, IC6G$1.C1-
- new net N$31: C29.1, IC6G$1.V+
- new net N$36: IC6G$1.R1IN, SV3.3
- new net N$38: IC6G$1.T1OUT, SV3.5
- new net N$39: IC6G$1.R2IN, SV3.2
- new net N$40: C30.1, IC6G$1.V-
- new net N$41: IC7G$1.T2OUT, SV1.4
- new net RTS1_TTL: IC2G$1.OP0, IC7G$1.T2IN
- new net RTS2_TTL: IC2G$1.OP1, IC6G$1.T2IN
- new net RXD2_TTL: IC2G$1.RXDB, IC6G$1.R1OUT
- new net TXD2_TTL: IC2G$1.TXDB, IC6G$1.T1IN
- net GND: now also C30.2, SV1.9, SV3.9; no longer X1.5
- net N$18: now also SV1.5; no longer X1.3
- net N$28: now also SV1.2; no longer X1.8
- net N$8: now also SV1.3; no longer X1.2
- net VCC: now also C29.2

Commit message: I/O board (Ultra version) bug fixes
Parts:
- removed LED1: (no value), led:LED5MM
- added C31: 100N, rcl:C-EUC0603
- added IC8: 74LVC1G04DBV, 74xx-little-us:74LVC1G04DBV
- added JP1: (no value), pinhead:PINHD-1X2
- R13: device rcl:R-EU_0204/5 -> rcl:R-EU_0204/7
Connections:
- removed net N$28: IC7G$1.R2IN, SV1.2
- removed net N$41: IC7G$1.T2OUT, SV1.4
- new net COM1_CTS: IC7G$1.R2IN, SV1.8
- new net COM1_RXD: IC7G$1.R1IN, SV1.1
- new net COM1_TXD: IC7G$1.T1OUT, SV1.3
- net GND: now also C31.2, SV1.5, SV3.5; no longer SV1.9, SV3.9
- net N$15: now also SV3.7; no longer SV3.4
- net N$18: now also IC7G$1.T2OUT, SV1.7; no longer IC7G$1.T1OUT, SV1.5
- net N$33: now also JP1.2; no longer LED1.C
- net N$34: now also JP1.1; no longer LED1.A
- net N$36: now also SV3.1; no longer SV3.3
- net N$38: now also SV3.3; no longer SV3.5
- net N$39: now also SV3.8; no longer SV3.2
- net N$8: now also IC2G$1.IRQ, IC8A.I, R13.1; no longer IC7G$1.R1IN, SV1.3
- net UART_RX_IRQ: now also IC8A.O; no longer IC2G$1.IRQ, R13.1
- net VCC: now also C31.1
Other:
- moved on the sheet: C1, C10, C12, C14, C15, C16, C17, C19, C2, C21, C24, C26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
